Commit message: update Gazebo

File: 6.ws_simulations/src/mycar_description/urdf/urdf/CyberNaviRobot.urdf (robot description, URDF)
Before this commit: robot CyberNaviRobot, 5 links, 4 joints
Links:
- added link camera, mass 0.1; collision box size=0.05 0.05 0.05; visual box size=0.05 0.05 0.05
- added link depth_camera, mass 0.1; collision box size=0.05 0.05 0.05; visual box size=0.05 0.05 0.05
- added link laser, mass 0.1; collision box size=0.05 0.05 0.05; visual box size=0.05 0.05 0.05
Joints:
- added joint camera_joint: type fixed, parent base_link, child camera, origin xyz=0.2 0 0.15 rpy=0 0 0
- added joint depth_camera_joint: type fixed, parent base_link, child depth_camera, origin xyz=0.2 0 0.2 rpy=0 0 0
- added joint laser_joint: type fixed, parent base_link, child laser, origin xyz=0.2 0 0.1 rpy=0 0 0
